Commit message: changing the mass of all component and inertia of left and right front wheel

File: urdf/robot.xacro (robot description, xacro)
@@ -12,7 +12,7 @@
       <origin xyz="0.0 0 0.05" rpy="0 0 0"/>
       <inertia
-          ixx="7.27e-3" ixy="0" ixz="0"
-          iyy="7.95e-3" iyz="0"
-          izz="7.35e-3"
+          ixx="0.00727" ixy="0" ixz="0"
+          iyy="0.00795" iyz="0"
+          izz="0.00735"
       />
     </inertial>
@@ -52,10 +52,10 @@
     </visual>
     <inertial>
-      <mass value="4"/>
+      <mass value="0.4"/>
       <origin xyz="0 0 0" rpy="0 0 0"/>
       <inertia
-          ixx="1.0" ixy="0" ixz="0"
-          iyy="1.0" iyz="0"
-          izz="1.0"
+          ixx="0.000213" ixy="0" ixz="0"
+          iyy="0.000213" iyz="0"
+          izz="0.00032"
       />
     </inertial>
@@ -77,5 +77,5 @@
     <inertial>
       <origin xyz="0 0 0" rpy="0 1.5707 1.5707"/>
-      <mass value="2"/>
+      <mass value="0.2"/>
       <inertia
         ixx="1.0" ixy="0.0" ixz="0.0"
@@ -108,5 +108,5 @@
     <inertial>
       <origin xyz="0 0 0" rpy="0 1.5707 1.5707"/>
-      <mass value="2"/>
+      <mass value="0.2"/>
       <inertia
         ixx="1.0" ixy="0.0" ixz="0.0"
@@ -138,10 +138,10 @@
     </visual>
     <inertial>
-      <mass value="4"/>
-      <origin xyz="0.0 0 0.0" rpy="0 0 0"/>
-      <inertia
-          ixx="1.0" ixy="0" ixz="0"
-          iyy="1.0" iyz="0"
-          izz="1.0"
+      <mass value="0.4"/>
+      <origin xyz="0 0 0" rpy="0 0 0"/>
+      <inertia
+          ixx="0.000213" ixy="0" ixz="0"
+          iyy="0.000213" iyz="0"
+          izz="0.00032"
       />
     </inertial>
@@ -163,5 +163,5 @@
     <inertial>
       <origin xyz="0 0 0" rpy="0 1.5707 1.5707"/>
-      <mass value="2"/>
+      <mass value="0.2"/>
       <inertia
         ixx="1.0" ixy="0.0" ixz="0.0"
@@ -194,5 +194,5 @@
     <inertial>
       <origin xyz="0 0 0" rpy="0 1.5707 1.5707"/>
-      <mass value="2"/>
+      <mass value="0.2"/>
       <inertia
         ixx="1.0" ixy="0.0" ixz="0.0"
